Commit message: Remove the angle limit for wheel [bugfix], and add the ctrl.py(still have some bug to fix)

File: resources/robots/diablo_plus/urdf/diablo_plus.urdf (robot description, URDF)
Before this commit: robot diablo_plus, 7 links, 6 joints
Joints:
- joint left_wheel_joint: limit lower=-3.14 upper=3.14 effort=20 velocity=30 -> effort=20 velocity=30
- joint right_wheel_joint: limit lower=-3.14 upper=3.14 effort=20 velocity=30 -> effort=20 velocity=30

Commit message: Transform the wheel collision to cylinder

File: resources/robots/diablo_plus/urdf/diablo_plus.urdf (robot description, URDF)
Before this commit: robot diablo_plus, 7 links, 6 joints
Links:
- link left_wheel: geometry collision cylinder length=0.035 radius=0.085; visual mesh filename=../meshes/left_wheel.STL
- link right_wheel: geometry collision cylinder length=0.035 radius=0.085; visual mesh filename=../meshes/right_wheel.STL

Commit message: remake the diablo_plus urdf

File: resources/robots/diablo_plus/urdf/diablo_plus.urdf (robot description, URDF)
Before this commit: robot diablo_plus, 7 links, 6 joints
Links:
- link right_knee: mass 0.149174408983867 -> 2.0
Joints:
- joint left_wheel_joint: origin xyz=0.16611 0.01266 -0.11138 rpy=0 0 0 -> xyz=0.16611 0.02266 -0.11138 rpy=0 0 0
- joint right_wheel_joint: origin xyz=0.16601 -0.01796 -0.11022 rpy=0 0 0 -> xyz=0.1666 -0.03046 -0.11066 rpy=0 0 0

Commit message: ctrl.py is okay to use now

File: resources/robots/diablo_plus/urdf/diablo_plus.urdf (robot description, URDF)
Before this commit: robot diablo_plus2, 7 links, 6 joints
Links:
- link left_wheel: geometry collision mesh filename=../meshes/left_wheel.STL; visual mesh filename=../meshes/left_wheel.STL
- link right_wheel: geometry collision mesh filename=../meshes/right_wheel.STL; visual mesh filename=../meshes/right_wheel.STL

Commit message: add cylinder collision of wheels and Instruction of RL

File: resources/robots/diablo_plus/urdf/diablo_plus.urdf (robot description, URDF)
Before this commit: robot diablo_plus2, 7 links, 6 joints
Links:
- link left_wheel: geometry collision cylinder length=0.05 radius=0.086; visual mesh filename=../meshes/left_wheel.STL
- link right_wheel: geometry collision cylinder length=0.05 radius=0.086; visual mesh filename=../meshes/right_wheel.STL

Commit message: urdf tunning and the init angle tuning

File: resources/robots/diablo_plus/urdf/diablo_plus.urdf (robot description, URDF)
Before this commit: robot diablo_plus2, 7 links, 6 joints
Links:
- link left_wheel: geometry collision cylinder length=0.035 radius=0.086; visual mesh filename=../meshes/left_wheel.STL
- link right_wheel: geometry collision cylinder length=0.035 radius=0.086; visual mesh filename=../meshes/right_wheel.STL
