Commit message: add diablo_plus_pro urdf (big wheel)

File: resources/robots/diablo_plus_pro/urdf/diablo_plus_pro.urdf (robot description, URDF)
Before this commit: robot diablo_plus2, 7 links, 6 joints
Links:
- removed link left_hip
- removed link left_knee
- removed link left_wheel
- removed link right_hip
- removed link right_knee
- removed link right_wheel
- added link left_hip_link, mass 2.0; collision mesh filename=package://diablo_plus_pro/meshes/left_hip_link.STL; visual mesh filename=package://diablo_plus_pro/meshes/left_hip_link.STL
- added link left_knee_link, mass 2.0; collision mesh filename=package://diablo_plus_pro/meshes/left_knee_link.STL; visual mesh filename=package://diablo_plus_pro/meshes/left_knee_link.STL
- added link left_wheel_link, mass 2.0; collision mesh filename=package://diablo_plus_pro/meshes/left_wheel_link.STL; visual mesh filename=package://diablo_plus_pro/meshes/left_wheel_link.STL
- added link right_hip_link, mass 2.0; collision mesh filename=package://diablo_plus_pro/meshes/right_hip_link.STL; visual mesh filename=package://diablo_plus_pro/meshes/right_hip_link.STL
- added link right_knee_link, mass 2.0; collision mesh filename=package://diablo_plus_pro/meshes/right_knee_link.STL; visual mesh filename=package://diablo_plus_pro/meshes/right_knee_link.STL
- added link right_wheel_link, mass 2.00; collision mesh filename=package://diablo_plus_pro/meshes/right_wheel_link.STL; visual mesh filename=package://diablo_plus_pro/meshes/right_wheel_link.STL
- link base_link: geometry collision mesh filename=package://diablo_plus_pro/meshes/base_link.STL; visual mesh filename=package://diablo_plus_pro/meshes/base_link.STL
Joints:
- joint left_hip_joint: child left_hip -> left_hip_link
- joint left_knee_joint: child left_knee -> left_knee_link; origin xyz=-0.15051 0.11148 -0.1317 rpy=0 0 0 -> xyz=-0.088027 0.11148 -0.17958 rpy=0 0 0; parent left_hip -> left_hip_link
- joint left_wheel_joint: child left_wheel -> left_wheel_link; limit effort=20 velocity=30 -> lower=0 upper=0 effort=20 velocity=30; origin xyz=0.16611 0.02266 -0.11138 rpy=0 0 0 -> xyz=0.17064 0.02266 0.10432 rpy=0 0 0; parent left_knee -> left_knee_link
- joint right_hip_joint: child right_hip -> right_hip_link
- joint right_knee_joint: child right_knee -> right_knee_link; origin xyz=-0.15071 -0.10364 -0.13147 rpy=0 0 0 -> xyz=-0.088029 -0.10364 -0.17958 rpy=0 0 0; parent right_hip -> right_hip_link
- joint right_wheel_joint: child right_wheel -> right_wheel_link; limit effort=20 velocity=30 -> lower=0 upper=0 effort=20 velocity=30; origin xyz=0.1666 -0.03046 -0.11066 rpy=0 0 0 -> xyz=0.17064 -0.03046 0.10432 rpy=0 0 0; parent right_knee -> right_knee_link

Commit message: run not so bad, still have some to fix

File: resources/robots/diablo_plus_pro/urdf/diablo_plus_pro.urdf (robot description, URDF)
Before this commit: robot diablo_plus_pro, 7 links, 6 joints
Links:
- link base_link: geometry collision mesh filename=../meshes/base_link.STL; visual mesh filename=../meshes/base_link.STL
- link left_hip_link: geometry collision mesh filename=../meshes/left_hip_link.STL; visual mesh filename=../meshes/left_hip_link.STL
- link left_knee_link: geometry collision mesh filename=../meshes/left_knee_link.STL; visual mesh filename=../meshes/left_knee_link.STL
- link left_wheel_link: geometry collision cylinder length=0.035 radius=0.16; visual mesh filename=../meshes/left_wheel_link.STL
- link right_hip_link: geometry collision mesh filename=../meshes/right_hip_link.STL; visual mesh filename=../meshes/right_hip_link.STL
- link right_knee_link: geometry collision mesh filename=../meshes/right_knee_link.STL; visual mesh filename=../meshes/right_knee_link.STL
- link right_wheel_link: geometry collision cylinder length=0.035 radius=0.16; visual mesh filename=../meshes/right_wheel_link.STL
Joints:
- joint left_hip_joint: limit lower=-3.14 upper=3.14 effort=100 velocity=10 -> lower=-1.0 upper=1.2 effort=80 velocity=15
- joint left_knee_joint: limit lower=-3.14 upper=3.14 effort=100 velocity=10 -> lower=0 upper=1.6 effort=80 velocity=15
- joint left_wheel_joint: limit lower=0 upper=0 effort=20 velocity=30 -> effort=20 velocity=30
- joint right_hip_joint: limit lower=-3.14 upper=3.14 effort=100 velocity=10 -> lower=-1.0 upper=1.2 effort=80 velocity=15
- joint right_knee_joint: limit lower=-3.14 upper=3.14 effort=100 velocity=10 -> lower=0 upper=1.6 effort=80 velocity=15
- joint right_wheel_joint: limit lower=0 upper=0 effort=20 velocity=30 -> effort=20 velocity=30

Commit message: 直接把pro的模型放在了plus的config里面，结果terrain突破7，不知道怎么做到的，现在在比对两份config的区别

File: resources/robots/diablo_plus_pro/urdf/diablo_plus_pro.urdf (robot description, URDF)
Before this commit: robot diablo_plus_pro, 7 links, 6 joints
Joints:
- joint left_knee_joint: limit lower=0 upper=1.6 effort=80 velocity=15 -> lower=0 upper=1.20 effort=80 velocity=15
- joint right_knee_joint: limit lower=0 upper=1.6 effort=80 velocity=15 -> lower=0 upper=1.20 effort=80 velocity=15
